File: KiCad/io_coupling_MCU_enhanced/io_coupling_MCU_enhanced.kicad_pcb (KiCad board)
At the start: 4 copper layers, 72.8 x 82.1 mm, 76 parts, among them IC1 AP63205, IC2 AP2112K-3.3TRG1, J10 10PIN_HEADER, J2 Conn_Coaxial, J3 1987724, J4 1987724, J5 1987724, J6 1987724, J7 10PIN_HEADER, J8 10PIN_HEADER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

Commit message: updated comment on pcb
Other:
- board text added: "Order Impedance Controlled JLC04161H-7628 (0.35mm ANT trace width corresponds to this)"
- board text removed: "Order Impedance Controlled JLC04161H-7628 (0.3mm ANT trace width corresponds to this)"
Changed lines of the file:
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@@
     (effects (font (size 1 1) (thickness 0.15)))
   )
-  (gr_text "Order Impedance Controlled JLC04161H-7628\n(0.3mm ANT trace width corresponds to this)" (at -4.8 -32.7) (layer "Cmts.User")
+  (gr_text "Order Impedance Controlled JLC04161H-7628\n(0.35mm ANT trace width corresponds to this)" (at -4.8 -32.7) (layer "Cmts.User")
     (effects (font (size 0.2 0.2) (thickness 0.05) bold) (justify left bottom))
   )
